File: Kicad_PCBs/MegaShield/MegaShield.kicad_pcb (KiCad board)
At the start: 2 copper layers, 95 x 110 mm, 22 parts, among them J1 rs485conn, J10 limitSwitches, J11 tmc2208, J12 GND_VIN, J2 Ypow, J3 rs485conn, J4 5V_VIN, J5 HeatingPad, J6 Xpow, J7 12V_VIN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

Commit message: Updated bunch of stuff
Parts:
- removed J12: GND_VIN, Quickprints:VinPad
- removed J4: 5V_VIN, Quickprints:VinPad
- C1: value CAP -> 47u
- J5: value HeatingPad -> HeatingOut
- M1: value MPMOS -> FQP27P06
- Q1: value 2N2219 -> 2N3904
- R1: value R -> 10k
- R2: value R -> 1k
